File: beehive-monitor.kicad_sch (KiCad schematic)
At the start: 4 parts, among them J1 CONSMA002-L-G, J2 Conn_ARM_JTAG_SWD_10, J3 643270100308, U1 RAK3172

Commit message: Board
Parts:
- added J4, J5: Conn_02x08_Odd_Even, Connector_PinHeader_2.54mm:PinHeader_2x08_P2.54mm_Horizontal, symbol Connector_Generic:Conn_02x08_Odd_Even
Connections:
- net GND: now also J4.12 (Pin_12), J4.16 (Pin_16), J4.4 (Pin_4), J4.8 (Pin_8), J5.12 (Pin_12), J5.16 (Pin_16), J5.4 (Pin_4), J5.8 (Pin_8)
- net NAU7802_SDIO: now reaches U1.10 (PA11/I2C_SDA)
- net LC_SELECTOR_00: now reaches U1.29 (PA0)
- net LC_SELECTOR_02: now reaches U1.3 (PA15/PIN_A4)
- net LC_SELECTOR_01: now reaches U1.6 (PA1)
- net NAU7802_SCK: now reaches U1.9 (PA12/I2C_SCL)
- new net LC_01_EXC_POS: J4.3 (Pin_3)
- new net LC_01_SIGNAL_A: J4.2 (Pin_2)
- new net LC_01_SIGNAL_B: J4.1 (Pin_1)
- new net LC_02_EXC_POS: J4.7 (Pin_7)
- new net LC_02_SIGNAL_A: J4.6 (Pin_6)
- new net LC_02_SIGNAL_B: J4.5 (Pin_5)
- new net LC_03_EXC_POS: J4.11 (Pin_11)
- new net LC_03_SIGNAL_A: J4.10 (Pin_10)
- new net LC_03_SIGNAL_B: J4.9 (Pin_9)
- new net LC_04_EXC_POS: J4.15 (Pin_15)
- new net LC_04_SIGNAL_A: J4.14 (Pin_14)
- new net LC_04_SIGNAL_B: J4.13 (Pin_13)
- new net LC_05_EXC_POS: J5.3 (Pin_3)
- new net LC_05_SIGNAL_A: J5.2 (Pin_2)
- new net LC_05_SIGNAL_B: J5.1 (Pin_1)
- new net LC_06_EXC_POS: J5.7 (Pin_7)
- new net LC_06_SIGNAL_A: J5.6 (Pin_6)
- new net LC_06_SIGNAL_B: J5.5 (Pin_5)
- new net LC_07_EXC_POS: J5.11 (Pin_11)
- new net LC_07_SIGNAL_A: J5.10 (Pin_10)
- new net LC_07_SIGNAL_B: J5.9 (Pin_9)
- new net LC_08_EXC_POS: J5.15 (Pin_15)
- new net LC_08_SIGNAL_A: J5.14 (Pin_14)
- new net LC_08_SIGNAL_B: J5.13 (Pin_13)
Other:
- added sheet LoadCells (LoadCells.kicad_sch)
- added sheet LoadCellsExcitationMux (LoadCellsExcitationMux.kicad_sch)
- moved on the sheet: J3
